Commit message: update apriltag tags.ymal and settings.yaml, update mapping in continuous_detection for images and camera_info, update urdf to include camera (but need to update with correct information in the link

File: catkin_ws/src/turtlebot3_description/urdf/turtlebot3_burger.urdf.xacro (robot description, xacro)
@@ -9,4 +9,34 @@
     <origin xyz="0.0 0.0 0.010" rpy="0 0 0"/>
   </joint>
+  <joint name="camera" type="fixed">
+    <parent link="base_footprint"/>
+    <child link="raspicam"/>
+    <origin
+      xyz="0.0 0.0 0.02"
+      rpy="0 0 1.77245385091"
+    />
+  </joint>
+  <link name="raspicam">
+    <visual>
+      <origin xyz="-0.032 0 0.0" rpy="0 0 0"/>
+      <geometry>
+        <mesh filename="package://turtlebot3_description/meshes/bases/burger_base.stl" scale="0.001 0.001 0.001"/>
+      </geometry>
+      <material name="light_black"/>
+    </visual>
+    <collision>
+      <origin xyz="-0.032 0 0.070" rpy="0 0 0"/>
+      <geometry>
+        <box size="0.140 0.140 0.143"/>
+      </geometry>
+    </collision>
+    <inertial>
+      <origin xyz="0 0 0" rpy="0 0 0"/>
+      <mass value="8.2573504e-01"/>
+      <inertia ixx="2.2124416e-03" ixy="-1.2294101e-05" ixz="3.4938785e-05"
+               iyy="2.1193702e-03" iyz="-5.0120904e-06"
+               izz="2.0064271e-03" />
+    </inertial>
+  </link>
   <link name="base_link">
     <visual>

Commit message: update the raspicam in the urdf file with proper box size, and approximate orientation and position

File: catkin_ws/src/turtlebot3_description/urdf/turtlebot3_burger.urdf.xacro (robot description, xacro)
@@ -13,29 +13,15 @@
     <child link="raspicam"/>
     <origin
-      xyz="0.0 0.0 0.02"
-      rpy="0 0 1.77245385091"
+      xyz="0.0172 0.0 0.15"
+      rpy="${-pi/2} 0 ${-pi/2}"
     />
   </joint>
   <link name="raspicam">
-    <visual>
-      <origin xyz="-0.032 0 0.0" rpy="0 0 0"/>
+    <collision>
+      <origin xyz="0 0 0 0" rpy="0 0 0"/>
       <geometry>
-        <mesh filename="package://turtlebot3_description/meshes/bases/burger_base.stl" scale="0.001 0.001 0.001"/>
-      </geometry>
-      <material name="light_black"/>
-    </visual>
-    <collision>
-      <origin xyz="-0.032 0 0.070" rpy="0 0 0"/>
-      <geometry>
-        <box size="0.140 0.140 0.143"/>
+        <box size="0.025 0.024 0.009"/>
       </geometry>
     </collision>
-    <inertial>
-      <origin xyz="0 0 0" rpy="0 0 0"/>
-      <mass value="8.2573504e-01"/>
-      <inertia ixx="2.2124416e-03" ixy="-1.2294101e-05" ixz="3.4938785e-05"
-               iyy="2.1193702e-03" iyz="-5.0120904e-06"
-               izz="2.0064271e-03" />
-    </inertial>
   </link>
   <link name="base_link">

Commit message: add the search and rescue node

File: catkin_ws/src/turtlebot3_description/urdf/turtlebot3_burger.urdf.xacro (robot description, xacro)
@@ -132,9 +132,9 @@
     <parent link="base_link"/>
     <child link="base_scan"/>
-    <origin xyz="-0.032 0 0.172" rpy="0 0 0"/>
+    <origin xyz="-0.032 0 0.172" rpy="0 0 ${pi}"/>
   </joint>
   <link name="base_scan">
     <visual>
-      <origin xyz="0 0 0.0" rpy="0 0 0"/>
+	<origin xyz="0 0 0.0" rpy="0 0 ${pi}"/>
       <geometry>
         <mesh filename="package://turtlebot3_description/meshes/sensors/lds.stl" scale="0.001 0.001 0.001"/>
